File: _autosave-KAPTON HEATER.kicad_sch (KiCad schematic)
At the start: 29 parts, among them J1 Conector, Q2 NTMFS4C10N

Commit message: formatted
Parts:
- removed F1, F2: Fuse, symbol Device:Fuse
Connections:
- net at U4.7~9 (+V): now also J1.1 (Pin_1)
Other:
- company: (none) -> QRET
- title: (none) -> Kapton PCB Heater
- moved on the sheet: CF1, Cin1, Cout1, J1, Q2, R1, R2, R3, R4, R5, TH1, TH2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
